File: EAGLE/projects/Balloon Project/Gondola_Sail_electronics_M4.sch (EAGLE design)
At the start: 28 parts

Commit message: derp
Parts:
- added R5, R6: ERA-3AEB104V, ERA-3AEB104V:ERA-3AEB104V
- added SD_POWER1: 3.3V_NCH_FET, Adafruit_Arduino:3.3V_NCH_FET
Connections:
- new net CUTDOWN: R5.1, SD_POWER1.G
- new net N$3: R6.2, SD_POWER1.S
- net REG_GND: now also R5.2, R6.1
Changed lines of the file:
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@@
 <?xml version="1.0" encoding="utf-8"?>
 <!DOCTYPE eagle SYSTEM "eagle.dtd">
-<eagle version="9.3.0">
+<eagle version="9.4.0">
 <drawing>
 <settings>
@@
 <part name="SJ3" library="jumper" library_urn="urn:adsk.eagle:library:252" deviceset="SJ" device="" package3d_urn="urn:adsk.eagle:package:15471/1"/>
 <part name="CUTDOWN" library="pinhead" library_urn="urn:adsk.eagle:library:325" deviceset="PINHD-1X2" device="/90" package3d_urn="urn:adsk.eagle:package:22437/2"/>
+<part name="SD_POWER1" library="Adafruit_Arduino" deviceset="3.3V_NCH_FET" device=""/>
+<part name="R5" library="ERA-3AEB104V" deviceset="ERA-3AEB104V" device=""/>
+<part name="R6" library="ERA-3AEB104V" deviceset="ERA-3AEB104V" device=""/>
 </parts>
 <sheets>
@@
 <attribute name="NAME" x="-82.55" y="78.105" size="1.778" layer="95" rot="R180"/>
 <attribute name="VALUE" x="-82.55" y="88.9" size="1.778" layer="96" rot="R180"/>
+</instance>
+<instance part="SD_POWER1" gate="G$1" x="195.58" y="50.8" smashed="yes" rot="R180">
+<attribute name="NAME" x="207.518" y="42.926" size="1.778" layer="95" rot="R180"/>
+</instance>
+<instance part="R5" gate="G$1" x="205.74" y="58.42" smashed="yes" rot="R90">
+<attribute name="NAME" x="209.55565" y="59.45918125" size="1.780640625" layer="95" rot="R180"/>
+</instance>
+<instance part="R6" gate="G$1" x="198.12" y="63.5" smashed="yes" rot="R180">
+<attribute name="NAME" x="196.84435" y="59.92081875" size="1.780640625" layer="95"/>
 </instance>
 </instances>
@@
 <label x="-134.62" y="-15.24" size="1.778" layer="95"/>
 </segment>
+<segment>
+<pinref part="R5" gate="G$1" pin="2"/>
+<wire x1="205.74" y1="63.5" x2="215.9" y2="63.5" width="0.1524" layer="91"/>
+<label x="205.74" y="63.5" size="1.778" layer="95"/>
+<pinref part="R6" gate="G$1" pin="1"/>
+<wire x1="203.2" y1="63.5" x2="205.74" y2="63.5" width="0.1524" layer="91"/>
+<junction x="205.74" y="63.5"/>
+</segment>
 </net>
 <net name="MCU_TX_3V" class="0">
@@
 </segment>
 </net>
+<net name="CUTDOWN" class="0">
+<segment>
+<pinref part="R5" gate="G$1" pin="1"/>
+<pinref part="SD_POWER1" gate="G$1" pin="G"/>
+<wire x1="205.74" y1="53.34" x2="205.74" y2="50.8" width="0.1524" layer="91"/>
+<wire x1="205.74" y1="50.8" x2="215.9" y2="50.8" width="0.1524" layer="91"/>
+<junction x="205.74" y="50.8"/>
+<label x="208.28" y="50.8" size="1.778" layer="95"/>
+</segment>
+</net>
+<net name="N$3" class="0">
+<segment>
+<pinref part="SD_POWER1" gate="G$1" pin="S"/>
+<pinref part="R6" gate="G$1" pin="2"/>
+<wire x1="190.5" y1="63.5" x2="193.04" y2="63.5" width="0.1524" layer="91"/>
+</segment>
+</net>

Commit message: update libraries
Parts:
- removed R6: ERA-3AEB104V, ERA-3AEB104V:ERA-3AEB104V
Connections:
- net N$3: no longer R6.2
- net REG_GND: no longer R6.1
Changed lines of the file:
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@@
 <?xml version="1.0" encoding="utf-8"?>
 <!DOCTYPE eagle SYSTEM "eagle.dtd">
-<eagle version="9.4.0">
+<eagle version="9.3.0">
 <drawing>
 <settings>
@@
 <part name="SD_POWER1" library="Adafruit_Arduino" deviceset="3.3V_NCH_FET" device=""/>
 <part name="R5" library="ERA-3AEB104V" deviceset="ERA-3AEB104V" device=""/>
-<part name="R6" library="ERA-3AEB104V" deviceset="ERA-3AEB104V" device=""/>
 </parts>
 <sheets>
@@
 <instance part="R5" gate="G$1" x="205.74" y="58.42" smashed="yes" rot="R90">
 <attribute name="NAME" x="209.55565" y="59.45918125" size="1.780640625" layer="95" rot="R180"/>
-</instance>
-<instance part="R6" gate="G$1" x="198.12" y="63.5" smashed="yes" rot="R180">
-<attribute name="NAME" x="196.84435" y="59.92081875" size="1.780640625" layer="95"/>
 </instance>
 </instances>
@@
 <wire x1="205.74" y1="63.5" x2="215.9" y2="63.5" width="0.1524" layer="91"/>
 <label x="205.74" y="63.5" size="1.778" layer="95"/>
-<pinref part="R6" gate="G$1" pin="1"/>
 <wire x1="203.2" y1="63.5" x2="205.74" y2="63.5" width="0.1524" layer="91"/>
 <junction x="205.74" y="63.5"/>
@@
 <segment>
 <pinref part="SD_POWER1" gate="G$1" pin="S"/>
-<pinref part="R6" gate="G$1" pin="2"/>
 <wire x1="190.5" y1="63.5" x2="193.04" y2="63.5" width="0.1524" layer="91"/>
 </segment>

Commit message: planning out pcb
placing parts and routing traces
added cutdown assembly
Parts:
- removed JP1, JP2: (no value), pinhead:PINHD-1X10/90
- removed JP3: (no value), pinhead:PINHD-1X5/90
- added ACC_PORT_1, ACC_PORT_2, ACC_PORT_3, ACC_PORT_4, ACC_PORT_5: (no value), pinhead:PINHD-1X5/90
- added C1: 10uF, SparkFun-Capacitors:10UF-POLAR-RADIAL-2.5MM-25V-20%
- added D1, D2: 1N4004, diode:1N4004
- added R6: RR0816P-103-D, 10K_SMD_resistors_RR0816p-103-D:RR0816P-103-D
- added REGULATOR_2_BATTERY_JUMPER: (no value), jumper:SJW
- added U$5: CUTDOWN_POWER_TRANSISTOR, Ultrasonic Misc PieceParts:CUTDOWN_POWER_TRANSISTOR
Connections:
- removed net N$3: SD_POWER1.S
- removed net N$4: CUTDOWN.1
- new net CUTDOWN_RETURN: CUTDOWN.1, U$5.D
- new net IMU_INT: ACC_PORT_3.1
- new net N$5: C1.+, R6.1, SD_POWER1.D, U$5.G
- net 3V: now also ACC_PORT_5.4; no longer JP3.2
- net 5V: now also ACC_PORT_5.5; no longer JP3.3
- net ACC_MCU_A0: now also ACC_PORT_2.5; no longer JP1.5
- net ACC_MCU_A1: now also ACC_PORT_2.4; no longer JP1.4
- net ACC_MCU_A5: now also ACC_PORT_2.3; no longer JP1.3
- net ADC_ALRT: now also ACC_PORT_3.4; no longer JP2.9
- net ALT_MISO: now also ACC_PORT_3.3; no longer JP2.8
- net BATT_GND: now also C1.-, R5.2, REGULATOR_2_BATTERY_JUMPER.1, SD_POWER1.S, U$5.S
- net BATT_VIN: now also R6.2
- net CUTDOWN: now also D1.C, D2.C
- net GPS_FIX_3V: now also ACC_PORT_2.2; no longer JP1.2
- net GPS_FIX_5V: now also ACC_PORT_2.1
- net GPS_PPS_5V: no longer JP1.1
- net I2C_SCL: now also ACC_PORT_1.2; no longer JP1.7
- net I2C_SDA: now also ACC_PORT_1.1; no longer JP1.6
- net IMU1_INT: no longer JP2.6
- net IMU1_PS0: now also ACC_PORT_4.5; no longer JP2.5
- net IMU1_PS1: now also ACC_PORT_4.4; no longer JP2.4
- net IMU1_RST: now also ACC_PORT_3.2; no longer JP2.7
- net MCU_AREF: now also ACC_PORT_4.2; no longer JP2.2
- net MCU_CUTDOWN: now also D1.A
- net MCU_EN: now also ACC_PORT_4.1; no longer JP2.1
- net MCU_RST: now also ACC_PORT_4.3; no longer JP2.3
- net MCU_SWCLK/RST: now also ACC_PORT_5.1; no longer JP3.4
- net MCU_SWDIO: now also ACC_PORT_5.2; no longer JP3.5
- net REG_GND: now also ACC_PORT_5.3, REGULATOR_2_BATTERY_JUMPER.2; no longer JP3.1, R5.2
- net SD_CD: now also ACC_PORT_3.5; no longer JP2.10
- net SPI_CLK: now also ACC_PORT_1.5; no longer JP1.10
- net SPI_MISO: now also ACC_PORT_1.4; no longer JP1.9
- net SPI_MOSI: now also ACC_PORT_1.3; no longer JP1.8
- net XBEE_CUTDOWN: now also D2.A
Other:
- note added: "SENSOR_PACK SCHEMATIC"
- moved on the sheet: ALT_POWER, BATT, CUTDOWN, IMU1_POWER, IMU2_2_MCU, IMU2_POWER, PITOT_2_MCU, R1, R2, R3, R4, R5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

Commit message: added minimal sensorpack
full sensor pack has too many breakout pins, need to trim down the size of the board. starting routing traces
Connections:
- removed net GPS_EN: U$8.4
- net GPS_EN_3V: now also U$8.4
Changed lines of the file:
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@@
 <label x="134.62" y="55.88" size="1.778" layer="95"/>
+</segment>
+<segment>
+<pinref part="U$8" gate="A" pin="4"/>
+<wire x1="166.37" y1="86.36" x2="166.37" y2="83.82" width="0.1524" layer="91"/>
+<wire x1="166.37" y1="83.82" x2="182.88" y2="83.82" width="0.1524" layer="91"/>
+<label x="177.8" y="83.82" size="1.778" layer="95"/>
 </segment>
 </net>
@@
 </segment>
 </net>
-<net name="GPS_EN" class="0">
-<segment>
-<pinref part="U$8" gate="A" pin="4"/>
-<wire x1="166.37" y1="86.36" x2="166.37" y2="83.82" width="0.1524" layer="91"/>
-<wire x1="166.37" y1="83.82" x2="182.88" y2="83.82" width="0.1524" layer="91"/>
-<label x="177.8" y="83.82" size="1.778" layer="95"/>
-</segment>
-</net>
