File: EAGLE/projects/Balloon Project/Gondola_Sail_electronics_M4_minimal.sch (EAGLE design)
At the start: 34 parts

Commit message: optimized board layout - finished
-minimized vias
-optimized some routes
-added silkscreen to xbee
-ERC and DRC checks out for all boards
-ready for ordering
Connections:
- net 5V: now also SERVO_CONTROL.2; no longer SERVO_CONTROL.3
- net RUDDER_SERVO_PWM_5V: now also SERVO_CONTROL.3; no longer SERVO_CONTROL.2
Changed lines of the file:
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@@
 </segment>
 <segment>
-<pinref part="SERVO_CONTROL" gate="A" pin="3"/>
-<wire x1="15.24" y1="128.27" x2="27.94" y2="128.27" width="0.1524" layer="91"/>
-<label x="25.4" y="128.27" size="1.778" layer="95"/>
+<pinref part="SERVO_CONTROL" gate="A" pin="2"/>
+<wire x1="15.24" y1="125.73" x2="27.94" y2="125.73" width="0.1524" layer="91"/>
+<label x="25.4" y="125.73" size="1.778" layer="95"/>
 </segment>
 </net>
@@
 </segment>
 <segment>
-<pinref part="SERVO_CONTROL" gate="A" pin="2"/>
-<wire x1="15.24" y1="125.73" x2="27.94" y2="125.73" width="0.1524" layer="91"/>
-<label x="25.4" y="125.73" size="1.778" layer="95"/>
+<pinref part="SERVO_CONTROL" gate="A" pin="3"/>
+<wire x1="15.24" y1="128.27" x2="27.94" y2="128.27" width="0.1524" layer="91"/>
+<label x="25.4" y="128.27" size="1.778" layer="95"/>
 </segment>
 </net>
@@
 </sheet>
 </sheets>
+<errors>
+</errors>
 </schematic>
 </drawing>
